File: full-size-sink/T430-pcie-sink.sch (KiCad schematic (older format))
At the start: 22 parts, among them J1 miniPCIe, J10 Conn_01x01, J11 Conn_01x01, J12 Conn_01x01, J13 Conn_01x01, J14 Conn_01x01, J15 Conn_01x01, J2 Conn_01x22_MountingPin, J3 Conn_01x24_MountingPin, J4 M.2-NGFF-A+E-Key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

Commit message: Add suspend oscillator
Seems to be mandatory in the NGFF M.2 spec
Parts:
- added C?: 100 nC, Capacitor_SMD:C_0805_2012Metric_Pad1.15x1.40mm_HandSolder, symbol Device:C
- added U?: DSC60XXB, microchip-lga:LGA4-1.6x1.2, symbol oscillator:DSC60XXB
Connections:
- net +3V3: now also C?.1, U?.1 (OE), U?.4 (VDD)
- net GND: now also C?.2, U?.2 (GND)
- net SUSCLK: now reaches J4.50 (SUSCLK)
- net SUSCLK: now also U?.3 (OUT)
Changed lines of the file:
@@
 $EndComp
 NoConn ~ 9300 5300
+$Comp
+L oscillator:DSC60XXB U?
+U 1 1 5DFD9B7B
+P 7900 5350
+F 0 "U?" H 7900 5715 50  0000 C CNN
+F 1 "DSC60XXB" H 7900 5624 50  0000 C CNN
+F 2 "microchip-lga:LGA4-1.6x1.2" H 7900 5300 50  0001 C CNN
+F 3 "" H 7900 5300 50  0001 C CNN
+	1    7900 5350
+	1    0    0    -1
+$EndComp
+$Comp
+L Device:C C?
+U 1 1 5DFDAF34
+P 8750 5500
+F 0 "C?" H 8865 5546 50  0000 L CNN
+F 1 "100 nC" H 8865 5455 50  0000 L CNN
+F 2 "Capacitor_SMD:C_0805_2012Metric_Pad1.15x1.40mm_HandSolder" H 8788 5350 50  0001 C CNN
+F 3 "~" H 8750 5500 50  0001 C CNN
+	1    8750 5500
+	1    0    0    -1
+$EndComp
+$Comp
+L power:+3V3 #PWR?
+U 1 1 5DFDB73B
+P 8750 5100
+F 0 "#PWR?" H 8750 4950 50  0001 C CNN
+F 1 "+3V3" H 8765 5273 50  0000 C CNN
+F 2 "" H 8750 5100 50  0001 C CNN
+F 3 "" H 8750 5100 50  0001 C CNN
+	1    8750 5100
+	1    0    0    -1
+$EndComp
+Wire Wire Line
+	8250 5250 8300 5250
+Wire Wire Line
+	8750 5250 8750 5100
+Wire Wire Line
+	8750 5250 8750 5350
+Connection ~ 8750 5250
+Wire Wire Line
+	8750 5650 8750 5750
+Wire Wire Line
+	8750 5750 7400 5750
+Wire Wire Line
+	7400 5750 7400 5450
+Wire Wire Line
+	7400 5450 7550 5450
+$Comp
+L power:GND #PWR?
+U 1 1 5E015C96
+P 7400 5850
+F 0 "#PWR?" H 7400 5600 50  0001 C CNN
+F 1 "GND" H 7405 5677 50  0000 C CNN
+F 2 "" H 7400 5850 50  0001 C CNN
+F 3 "" H 7400 5850 50  0001 C CNN
+	1    7400 5850
+	1    0    0    -1
+$EndComp
+Wire Wire Line
+	7400 5850 7400 5750
+Connection ~ 7400 5750
+Wire Wire Line
+	8250 5450 8600 5450
+Text Label 8600 5450 2    50   ~ 0
+SUSCLK
+Wire Wire Line
+	7550 5250 7400 5250
+Wire Wire Line
+	7400 5250 7400 4900
+Wire Wire Line
+	7400 4900 8300 4900
+Wire Wire Line
+	8300 4900 8300 5250
+Connection ~ 8300 5250
+Wire Wire Line
+	8300 5250 8750 5250
+Wire Wire Line
+	7850 2900 8600 2900
+Text Label 8600 2900 2    50   ~ 0
+SUSCLK
 $EndSCHEMATC
